File: MCP73834 Test/MCP73834 Test.kicad_sch (KiCad schematic)
At the start: 12 parts, among them U1 MCP73834-xxx-UN

Commit message: add pcb design and lcsc part numbers
Parts:
- removed BT1: Battery_Cell, symbol Device:Battery_Cell
- added J1, J3: Screw_Terminal_01x02, easyeda2kicad:CONN-TH_XY308-2.54-2P, symbol Connector:Screw_Terminal_01x02
- added J2, J4: Conn_01x02_Pin, easyeda2kicad:HDR-TH_2P-P2.54-V-M, symbol Connector:Conn_01x02_Pin
- C1, C3: footprint (none) -> easyeda2kicad:CAP-SMD_BD4.0-L4.3-W4.3-FD; LCSC (none) -> C41435083
- D1: value LED -> RED; footprint (none) -> easyeda2kicad:LED0805-RD_RED; LCSC (none) -> C965812
- D2: value LED -> GREEN; footprint (none) -> easyeda2kicad:LED0805-RD_GREEN; LCSC (none) -> C965815
- R1, R2: footprint (none) -> easyeda2kicad:R0805; LCSC (none) -> C105878
- R3: footprint (none) -> easyeda2kicad:R0805; LCSC (none) -> C114555
- R4: footprint (none) -> easyeda2kicad:R0805; LCSC (none) -> C865614
- R5: footprint (none) -> easyeda2kicad:R0805; LCSC (none) -> C114748
- TH2: value NTCLE100E3103 -> NTCS0805E3103JHT; footprint (none) -> easyeda2kicad:R0805; LCSC (none) -> C511025
Connections:
- net GND: now also J1.1 (Pin_1), J2.2 (Pin_2), J3.2 (Pin_2), J4.2 (Pin_2)
- net VBatt: now also J1.2 (Pin_2), J2.1 (Pin_1)
- net VDD: now also J3.1 (Pin_1), J4.1 (Pin_1)
