File: TPS62152 Test/TPS62152 Test.kicad_sch (KiCad schematic)
At the start: 17 parts, among them J1 Conn_01x02_Pin, J2 Conn_01x02_Pin, J3 Conn_01x02_Pin, J4 Conn_01x02_Socket, U1 TPS62152RGTR

Commit message: tidy up
Parts:
- removed H1, H2, H3, H4: MountingHole, MountingHole:ToolingHole_1.152mm, symbol Mechanical:MountingHole
- J4: footprint Connector_PinHeader_2.54mm:PinHeader_1x02_P2.54mm_Vertical -> Connector_PinSocket_2.54mm:PinSocket_1x02_P2.54mm_Vertical

Commit message: update part numbers
Parts:
- C3: LCSC C440198 -> C45783
- R1: LCSC C14675 -> C25803
Changed lines of the file:
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@@
 			)
 		)
-		(property "LCSC" "C440198"
+		(property "LCSC" "C45783"
 			(at 165.1 93.98 0)
 			(effects
@@
 			)
 		)
-		(property "LCSC" "C14675"
+		(property "LCSC" "C25803"
 			(at 105.41 93.98 90)
 			(effects
